File: ShieldPCB_kicad/ShieldPCB.sch (KiCad schematic (older format))
At the start: 118 parts, among them J1 SECURED MODE, J10 PWM, J11 PWM, J12 COM, J13 LIGHTS, J14 PWR, J15 MOV, J16 PWR, J17 PWR, J18 MOV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

Commit message: PCB Shield finished and some changes in Qt software.
Parts:
- removed J22: LED, symbol HEADER_2
- removed Q1: MBT2222A, symbol NPN
- added C27, C28: 1uF, symbol CAP_NP
- added D1, D2, D3, D4: LED, symbol LED
- added D5: S2A, symbol DIODE
- added J22: EXP, symbol HEADER_6
- added J25: PWR, symbol HEADER_2
- added J26: DIG2, symbol HEADER_10
- added J27: DIG1, symbol HEADER_10
- added J28: EX, symbol HEADER_2
- added J29: BAT, symbol HEADER_2
- added J30: C, symbol HEADER_3
- added P1: Power, symbol HEADER_3
- added R64, R65: 1K, symbol R
- added R66, R67, R68, R69, R70, R71: 470, symbol R
- added R72, R74: 50K, symbol R
- added R73, R75: 10K, symbol R
- added R76, R77, R78, R79: 330, symbol R
- J18: value MOV -> SWT
- R57: value 5K -> 1K
- R60: value 5K -> 2K
- R62: value 100 -> 1K
Connections:
- net labels added: D40, D41, D42, D43, Vbat, Vdc
- net labels removed: D21
- wire segments 385 -> 445
- no-connect marks 12 -> 10
Other:
- note removed: "LEDs\n"
- note removed: "Max = 8\n"
- moved on the sheet: J1, J2, J23, J24, J3, J8, J9
